File: Spaceport/23-24/PCBs/Unified Board/Unified_Board/Unified_Board.kicad_pcb (KiCad board)
At the start: 4 copper layers, 92 x 74.7 mm, 52 parts, among them J1 Screw_Terminal_01x02, J2 Serial2 Breakout, J3 I2C Breakout, J4 Serial1 Breakout, J5 Conn_01x05_Pin, J6 Conn_01x09_Pin, J7 Screw_Terminal_01x02, U1 BNO055, U2 MAX-M10S, Y1 32.768kHz

Commit message: Update Unified_Board.kicad_pcb
Parts:
- moved J6 99.4 mm to (106.7, 135.0), turned to 90 degrees
- moved J5 84.7 mm to (106.7, 109.6), turned to 90 degrees
- moved C8 70.1 mm to (62.4, 54.4)
- moved BZ1 54.6 mm to (191.4, 107.8)
- moved C5 45.1 mm to (178.6, 62.2)
- moved C6 45.1 mm to (178.6, 57.5)
- moved BT1 44.9 mm to (195.4, 78.2)
- moved C3 44.9 mm to (192.7, 62.9)
- moved C4 44.9 mm to (192.7, 58.2)
- moved C7 44.9 mm to (195.4, 78.5)
- moved C9 44.9 mm to (175.6, 83.3)
- moved D3 44.9 mm to (195.2, 73.7)
- moved D5 44.9 mm to (186.2, 66.7)
- moved R11 44.9 mm to (186.0, 70.5)
- moved R16 44.9 mm to (175.4, 75.5)
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Routing:
- net /Radio_RST: track 151.1 -> 0.00 mm
- net /Radio_INT: track 119.8 -> 0.00 mm
- net /SDA: track 170.9 -> 55.3 mm
- net /Radio_MISO: track 99.1 -> 0.00 mm
- net /Radio_MOSI: track 94.6 -> 0.00 mm
- net /SCL: track 150.0 -> 61.4 mm
- net /Radio_CS: track 85.9 -> 0.00 mm
- net /Radio_SCK: track 78.6 -> 0.00 mm
- net Net-(BZ1--): track 40.9 -> 3.00 mm
- net Net-(ANT1-RF_IN): track 31.5 -> 7.73 mm
- net GND: track 160.3 -> 145.3 mm
- net Net-(C12-Pad1): track 14.0 -> 0.00 mm
- net /Breakout_RX1: track 95.3 -> 85.2 mm
- net /Breakout_RX2: track 70.3 -> 60.7 mm
- net /Breakout_TX2: track 69.1 -> 60.3 mm
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Other:
- board text added: "Avionics Unified Board v1.2"
- board text removed: "Avionics Unified Board v1.1"
