File: Spaceport/23-24/PCBs/Unified Board/Unified_Board/Unified_Board.kicad_sch (KiCad schematic)
At the start: 51 parts, among them J1 Screw_Terminal_01x02, J2 Serial2 Breakout, J3 I2C Breakout, J4 Serial1 Breakout, J5 Conn_01x05_Pin, J6 Conn_01x09_Pin, U1 BNO055, U2 MAX-M10S, Y1 32.768kHz

Commit message: Fixed stage conditions
Parts:
- C12: value LP_C -> 10nF
- FB1: value LP_FerriteBead -> 68nH
- R16: value LP_R -> 10Ω
Changed lines of the file:
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@@
     (effects (font (size 1.27 1.27)) (justify left bottom))
-  )
-  (global_label "I2C Diagram" (shape input) (at 111.76 26.67 180) (fields_autoplaced)
-    (effects (font (size 1.27 1.27)) (justify right))
-    (property "Intersheetrefs" "${INTERSHEET_REFS}" (at 96.9216 26.67 0)
-      (effects (font (size 1.27 1.27)) (justify right) hide)
-    )
   )
   (symbol (lib_id "Connector:Screw_Terminal_01x02") (at 91.44 17.78 0) (unit 1)
@@
       (effects (font (size 1.27 1.27)) (justify left))
     )
-    (property "Value" "LP_FerriteBead" (at 231.14 44.3992 0)
+    (property "Value" "68nH" (at 231.14 44.3992 0)
       (effects (font (size 1.27 1.27)) (justify left))
     )
@@
       (effects (font (size 1.27 1.27)))
     )
-    (property "Value" "LP_C" (at 236.22 29.21 90)
+    (property "Value" "10nF" (at 236.22 29.21 90)
       (effects (font (size 1.27 1.27)))
     )
@@
       (effects (font (size 1.27 1.27)))
     )
-    (property "Value" "LP_R" (at 220.98 30.48 90)
-      (effects (font (size 1.27 1.27)))
-    )
+    (property "Value" "10Ω" (at 220.98 30.48 90)
+      (effects (font (size 1.27 1.27)))
+    )
